Commit message: Rename panda_arm.xacro -> arm.xacro
... and xacro:panda_arm -> xacro:arm
to be consistent with hand.xacro

File: franka_description/robots/arm.xacro (robot description, xacro)
@@ -3,5 +3,5 @@
   <!-- safety_distance: Minimum safety distance in [m] by which the collision volumes are expanded and which is enforced during robot motions -->
   <!-- arm_id: Namespace of the panda arm. Serves to differentiate between arms in case of multiple instances. -->
-  <xacro:macro name="panda_arm" params="arm_id:='panda' description_pkg:='franka_description' connected_to:='' xyz:='0 0 0' rpy:='0 0 0' safety_distance:=0">
+  <xacro:macro name="arm" params="arm_id:='panda' description_pkg:='franka_description' connected_to:='' xyz:='0 0 0' rpy:='0 0 0' safety_distance:=0">
     <xacro:unless value="${not connected_to}">
       <joint name="${arm_id}_joint_${connected_to}" type="fixed">

File: franka_description/robots/dual_panda_example.urdf.xacro (robot description, xacro)
@@ -3,5 +3,5 @@
   <xacro:arg name="arm_id_1" default="panda_1" />
   <xacro:arg name="arm_id_2" default="panda_2" />
-  <xacro:include filename="$(find franka_description)/robots/panda_arm.xacro"/>
+  <xacro:include filename="$(find franka_description)/robots/arm.xacro"/>
   <xacro:include filename="$(find franka_description)/robots/hand.xacro"/>
   <!-- box shaped table as base for the 2 Pandas -->
@@ -24,8 +24,8 @@
   </link>
   <!-- right arm with gripper -->
-  <xacro:panda_arm arm_id="$(arg arm_id_1)" connected_to="base"  xyz="0 -0.5 1" safety_distance="0.03"/>
+  <xacro:arm arm_id="$(arg arm_id_1)" connected_to="base"  xyz="0 -0.5 1" safety_distance="0.03"/>
   <xacro:hand ns="$(arg arm_id_1)" rpy="0 0 ${-pi/4}" connected_to="$(arg arm_id_1)_link8" safety_distance="0.03"/>
   <!-- left arm with gripper -->
-  <xacro:panda_arm arm_id="$(arg arm_id_2)" connected_to="base"  xyz="0 0.5 1" safety_distance="0.03"/>
+  <xacro:arm arm_id="$(arg arm_id_2)" connected_to="base"  xyz="0 0.5 1" safety_distance="0.03"/>
   <xacro:hand ns="$(arg arm_id_2)" rpy="0 0 ${-pi/4}" connected_to="$(arg arm_id_2)_link8" safety_distance="0.03"/>
 </robot>

File: franka_description/robots/panda_arm.urdf.xacro (robot description, xacro)
@@ -9,6 +9,6 @@
   <xacro:unless value="$(arg gazebo)">
     <!-- Create a URDF for a real hardware -->
-    <xacro:include filename="$(find franka_description)/robots/panda_arm.xacro" />
-    <xacro:panda_arm arm_id="$(arg arm_id)" safety_distance="0.03"/>
+    <xacro:include filename="$(find franka_description)/robots/arm.xacro" />
+    <xacro:arm arm_id="$(arg arm_id)" safety_distance="0.03" />
     <xacro:if value="$(arg hand)">
       <xacro:include filename="$(find franka_description)/robots/hand.xacro"/>
@@ -22,5 +22,5 @@
     <xacro:include filename="$(find franka_description)/robots/utils.xacro" />
     <xacro:include filename="$(find franka_description)/robots/panda_gazebo.xacro" />
-    <xacro:panda_arm arm_id="$(arg arm_id)" />
+    <xacro:arm arm_id="$(arg arm_id)" />
     <xacro:if value="$(arg hand)">
       <xacro:hand ns="$(arg arm_id)" rpy="0 0 ${-pi/4}" connected_to="$(arg arm_id)_link8" />

File: franka_description/robots/panda_gazebo.xacro (robot description, xacro)
@@ -10,5 +10,5 @@
   <!-- || Paolo Robuffo Giordano, Alessandro de Luca                || -->
   <!-- =============================================================== -->
-  <xacro:macro name="panda_arm" params="arm_id:='panda' connected_to:='' xyz:='0 0 0' rpy:='0 0 0'">
+  <xacro:macro name="arm" params="arm_id:='panda' connected_to:='' xyz:='0 0 0' rpy:='0 0 0'">
     <xacro:unless value="${not connected_to}">
       <joint name="${arm_id}_joint_${connected_to}" type="fixed">

Commit message: Use both, detailed meshes and coarse collision geometries
They serve different purposes:
- coarse collision geometries mimic the internal self-collision checking
  of the real-robot controller
- mesh models should be use for collision checking with environmental objects

File: franka_description/robots/arm.xacro (robot description, xacro)
@@ -11,10 +11,6 @@
       </joint>
     </xacro:unless>
-    <link name="${arm_id}_link0">
-      <visual>
-        <geometry>
-          <mesh filename="package://${description_pkg}/meshes/visual/link0.dae"/>
-        </geometry>
-      </visual>
+    <xacro:link arm_id="${arm_id}" name="link0">
+      <self_collision_geometries>
       <collision>
         <origin xyz="-0.075 0 0.06" rpy="0 ${pi/2} 0"/>
@@ -35,11 +31,8 @@
         </geometry>
       </collision>
-    </link>
-    <link name="${arm_id}_link1">
-      <visual>
-        <geometry>
-          <mesh filename="package://${description_pkg}/meshes/visual/link1.dae"/>
-        </geometry>
-      </visual>
+      </self_collision_geometries>
+    </xacro:link>
+    <xacro:link arm_id="${arm_id}" name="link1">
+      <self_collision_geometries>
       <collision>
         <origin xyz="0 0 -0.1915" rpy="0 0 0"/>
@@ -60,5 +53,6 @@
         </geometry>
       </collision>
-    </link>
+      </self_collision_geometries>
+    </xacro:link>
     <joint name="${arm_id}_joint1" type="revolute">
       <safety_controller k_position="100.0" k_velocity="40.0" soft_lower_limit="-2.8973" soft_upper_limit="2.8973"/>
@@ -69,10 +63,6 @@
       <limit effort="87" lower="-2.8973" upper="2.8973" velocity="2.1750"/>
     </joint>
-    <link name="${arm_id}_link2">
-      <visual>
-        <geometry>
-          <mesh filename="package://${description_pkg}/meshes/visual/link2.dae"/>
-        </geometry>
-      </visual>
+    <xacro:link arm_id="${arm_id}" name="link2">
+      <self_collision_geometries>
       <collision>
         <origin xyz="0 0 0" rpy="0 0 0"/>
@@ -93,5 +83,6 @@
         </geometry>
       </collision>
-    </link>
+      </self_collision_geometries>
+    </xacro:link>
     <joint name="${arm_id}_joint2" type="revolute">
       <safety_controller k_position="100.0" k_velocity="40.0" soft_lower_limit="-1.7628" soft_upper_limit="1.7628"/>
@@ -102,10 +93,6 @@
       <limit effort="87" lower="-1.7628" upper="1.7628" velocity="2.1750"/>
     </joint>
-    <link name="${arm_id}_link3">
-      <visual>
-        <geometry>
-          <mesh filename="package://${description_pkg}/meshes/visual/link3.dae"/>
-        </geometry>
-      </visual>
+    <xacro:link arm_id="${arm_id}" name="link3">
+      <self_collision_geometries>
       <collision>
         <origin xyz="0 0 -0.145" rpy="0 0 0"/>
@@ -126,5 +113,6 @@
         </geometry>
       </collision>
-    </link>
+      </self_collision_geometries>
+    </xacro:link>
     <joint name="${arm_id}_joint3" type="revolute">
       <safety_controller k_position="100.0" k_velocity="40.0" soft_lower_limit="-2.8973" soft_upper_limit="2.8973"/>
@@ -135,10 +123,6 @@
       <limit effort="87" lower="-2.8973" upper="2.8973" velocity="2.1750"/>
     </joint>
-    <link name="${arm_id}_link4">
-      <visual>
-        <geometry>
-          <mesh filename="package://${description_pkg}/meshes/visual/link4.dae"/>
-        </geometry>
-      </visual>
+    <xacro:link arm_id="${arm_id}" name="link4">
+      <self_collision_geometries>
       <collision>
         <origin xyz="0 0 0" rpy="0 0 0"/>
@@ -159,5 +143,6 @@
         </geometry>
       </collision>
-    </link>
+      </self_collision_geometries>
+    </xacro:link>
     <joint name="${arm_id}_joint4" type="revolute">
       <safety_controller k_position="100.0" k_velocity="40.0" soft_lower_limit="-3.0718" soft_upper_limit="-0.0698"/>
@@ -168,10 +153,6 @@
       <limit effort="87" lower="-3.0718" upper="-0.0698" velocity="2.1750"/>
     </joint>
-    <link name="${arm_id}_link5">
-      <visual>
-        <geometry>
-          <mesh filename="package://${description_pkg}/meshes/visual/link5.dae"/>
-        </geometry>
-      </visual>
+    <xacro:link arm_id="${arm_id}" name="link5">
+      <self_collision_geometries>
       <collision>
         <origin xyz="0 0 -0.26" rpy="0 0 0"/>
@@ -210,5 +191,6 @@
         </geometry>
       </collision>
-    </link>
+      </self_collision_geometries>
+    </xacro:link>
     <joint name="${arm_id}_joint5" type="revolute">
       <safety_controller k_position="100.0" k_velocity="40.0" soft_lower_limit="-2.8973" soft_upper_limit="2.8973"/>
@@ -219,10 +201,6 @@
       <limit effort="12" lower="-2.8973" upper="2.8973" velocity="2.6100"/>
     </joint>
-    <link name="${arm_id}_link6">
-      <visual>
-        <geometry>
-          <mesh filename="package://${description_pkg}/meshes/visual/link6.dae"/>
-        </geometry>
-      </visual>
+    <xacro:link arm_id="${arm_id}" name="link6">
+      <self_collision_geometries>
       <collision>
         <origin xyz="0 0 -0.03" rpy="0 0 0"/>
@@ -243,5 +221,6 @@
         </geometry>
       </collision>
-    </link>
+      </self_collision_geometries>
+    </xacro:link>
     <joint name="${arm_id}_joint6" type="revolute">
       <safety_controller k_position="100.0" k_velocity="40.0" soft_lower_limit="-0.0175" soft_upper_limit="3.7525"/>
@@ -252,10 +231,6 @@
       <limit effort="12" lower="-0.0175" upper="3.7525" velocity="2.6100"/>
     </joint>
-    <link name="${arm_id}_link7">
-      <visual>
-        <geometry>
-          <mesh filename="package://${description_pkg}/meshes/visual/link7.dae"/>
-        </geometry>
-      </visual>
+    <xacro:link arm_id="${arm_id}" name="link7">
+      <self_collision_geometries>
       <collision>
         <origin xyz="0 0 0.01" rpy="0 0 0"/>
@@ -276,5 +251,6 @@
         </geometry>
       </collision>
-    </link>
+      </self_collision_geometries>
+    </xacro:link>
     <joint name="${arm_id}_joint7" type="revolute">
       <safety_controller k_position="100.0" k_velocity="40.0" soft_lower_limit="-2.8973" soft_upper_limit="2.8973"/>

File: franka_description/robots/dual_panda_example.urdf.xacro (robot description, xacro)
@@ -25,7 +25,7 @@
   <!-- right arm with gripper -->
   <xacro:arm arm_id="$(arg arm_id_1)" connected_to="base"  xyz="0 -0.5 1" safety_distance="0.03"/>
-  <xacro:hand ns="$(arg arm_id_1)" rpy="0 0 ${-pi/4}" connected_to="$(arg arm_id_1)_link8" safety_distance="0.03"/>
+  <xacro:hand arm_id="$(arg arm_id_1)" rpy="0 0 ${-pi/4}" connected_to="$(arg arm_id_1)_link8" safety_distance="0.03"/>
   <!-- left arm with gripper -->
   <xacro:arm arm_id="$(arg arm_id_2)" connected_to="base"  xyz="0 0.5 1" safety_distance="0.03"/>
-  <xacro:hand ns="$(arg arm_id_2)" rpy="0 0 ${-pi/4}" connected_to="$(arg arm_id_2)_link8" safety_distance="0.03"/>
+  <xacro:hand arm_id="$(arg arm_id_2)" rpy="0 0 ${-pi/4}" connected_to="$(arg arm_id_2)_link8" safety_distance="0.03"/>
 </robot>

File: franka_description/robots/hand.urdf.xacro (robot description, xacro)
@@ -1,5 +1,6 @@
 <?xml version="1.0" encoding="utf-8"?>
 <robot xmlns:xacro="http://www.ros.org/wiki/xacro" name="hand">
+  <xacro:include filename="utils.xacro" />
   <xacro:include filename="hand.xacro"/>
-  <xacro:hand ns="panda" safety_distance="0.03"/>
+  <xacro:hand arm_id="panda" safety_distance="0.03"/>
 </robot>

File: franka_description/robots/hand.xacro (robot description, xacro)
@@ -2,18 +2,15 @@
 <robot xmlns:xacro="http://www.ros.org/wiki/xacro" name="hand">
   <!-- safety_distance: Minimum safety distance in [m] by which the collision volumes are expanded and which is enforced during robot motions -->
-  <xacro:macro name="hand" params="connected_to:='' ns:='' rpy:='0 0 0' xyz:='0 0 0' safety_distance:=0">
+  <!-- ns: used for joint and link names. Needed to distinguish joints and TFs in case of multiple arm instances. -->
+  <xacro:macro name="hand" params="connected_to:='' arm_id:='panda' rpy:='0 0 0' xyz:='0 0 0' safety_distance:=0 description_pkg:=franka_description">
     <xacro:unless value="${connected_to == ''}">
-      <joint name="${ns}_hand_joint" type="fixed">
+      <joint name="${arm_id}_hand_joint" type="fixed">
         <parent link="${connected_to}"/>
-        <child link="${ns}_hand"/>
+        <child link="${arm_id}_hand"/>
         <origin xyz="${xyz}" rpy="${rpy}"/>
       </joint>
     </xacro:unless>
-    <link name="${ns}_hand">
-      <visual>
-        <geometry>
-          <mesh filename="package://franka_description/meshes/visual/hand.dae"/>
-        </geometry>
-      </visual>
+    <xacro:link arm_id="${arm_id}" name="hand">
+      <self_collision_geometries>
       <collision>
         <origin xyz="0 0 0.04" rpy="0 ${pi/2} ${pi/2}"/>
@@ -52,13 +49,14 @@
         </geometry>
       </collision>
-    </link>
+      </self_collision_geometries>
+    </xacro:link>
     <!-- Define the hand_tcp frame -->
-    <link name="${ns}_hand_tcp" />
-    <joint name="${ns}_hand_tcp_joint" type="fixed">
+    <link name="${arm_id}_hand_tcp" />
+    <joint name="${arm_id}_hand_tcp_joint" type="fixed">
       <origin xyz="0 0 0.1034" rpy="0 0 0" />
-      <parent link="${ns}_hand" />
-      <child link="${ns}_hand_tcp" />
+      <parent link="${arm_id}_hand" />
+      <child link="${arm_id}_hand_tcp" />
     </joint>
-    <link name="${ns}_leftfinger">
+    <link name="${arm_id}_leftfinger">
       <visual>
         <geometry>
@@ -67,5 +65,5 @@
       </visual>
     </link>
-    <link name="${ns}_rightfinger">
+    <link name="${arm_id}_rightfinger">
       <visual>
         <origin xyz="0 0 0" rpy="0 0 ${pi}"/>
@@ -75,18 +73,18 @@
       </visual>
    </link>
-    <joint name="${ns}_finger_joint1" type="prismatic">
-      <parent link="${ns}_hand"/>
-      <child link="${ns}_leftfinger"/>
+    <joint name="${arm_id}_finger_joint1" type="prismatic">
+      <parent link="${arm_id}_hand"/>
+      <child link="${arm_id}_leftfinger"/>
       <origin xyz="0 0 0.0584" rpy="0 0 0"/>
       <axis xyz="0 1 0"/>
       <limit effort="100" lower="0.0" upper="0.04" velocity="0.2"/>
     </joint>
-    <joint name="${ns}_finger_joint2" type="prismatic">
-      <parent link="${ns}_hand"/>
-      <child link="${ns}_rightfinger"/>
+    <joint name="${arm_id}_finger_joint2" type="prismatic">
+      <parent link="${arm_id}_hand"/>
+      <child link="${arm_id}_rightfinger"/>
       <origin xyz="0 0 0.0584" rpy="0 0 0"/>
       <axis xyz="0 -1 0"/>
       <limit effort="100" lower="0.0" upper="0.04" velocity="0.2"/>
-      <mimic joint="${ns}_finger_joint1" />
+      <mimic joint="${arm_id}_finger_joint1" />
     </joint>
   </xacro:macro>

File: franka_description/robots/panda_arm.urdf.xacro (robot description, xacro)
@@ -9,9 +9,10 @@
   <xacro:unless value="$(arg gazebo)">
     <!-- Create a URDF for a real hardware -->
+    <xacro:include filename="utils.xacro" />
     <xacro:include filename="arm.xacro" />
     <xacro:arm arm_id="$(arg arm_id)" safety_distance="0.03" />
     <xacro:if value="$(arg hand)">
       <xacro:include filename="hand.xacro"/>
-      <xacro:hand ns="$(arg arm_id)" rpy="0 0 ${-pi/4}" connected_to="$(arg arm_id)_link8" safety_distance="0.03"/>
+      <xacro:hand arm_id="$(arg arm_id)" rpy="0 0 ${-pi/4}" connected_to="$(arg arm_id)_link8" safety_distance="0.03"/>
     </xacro:if>
   </xacro:unless>
@@ -24,5 +25,5 @@
     <xacro:arm arm_id="$(arg arm_id)" />
     <xacro:if value="$(arg hand)">
-      <xacro:hand ns="$(arg arm_id)" rpy="0 0 ${-pi/4}" connected_to="$(arg arm_id)_link8" />
+      <xacro:hand arm_id="$(arg arm_id)" rpy="0 0 ${-pi/4}" connected_to="$(arg arm_id)_link8" />
       <xacro:gazebo-joint joint="$(arg arm_id)_finger_joint1" transmission="hardware_interface/EffortJointInterface" />
       <xacro:gazebo-joint joint="$(arg arm_id)_finger_joint2" transmission="hardware_interface/EffortJointInterface" />

File: franka_description/robots/utils.xacro (robot description, xacro)
@@ -1,4 +1,38 @@
 <?xml version="1.0"?>
 <robot xmlns:xacro="http://www.ros.org/wiki/xacro">
+  <!-- ========================================================== -->
+  <!-- Macro to add a single link, both with                      -->
+  <!--  * detailed meshes for environmental collision checking    -->
+  <!--  * and coarse geometry models for self-collision checking  -->
+  <!--                                                            -->
+  <!-- name:  Name of the robot link (without prefix)             -->
+  <!-- self_collision_geometries:  self <collision> models        -->
+  <!-- ========================================================== -->
+  <xacro:macro name="link" params="arm_id name **self_collision_geometries">
+    <!-- sub-link defining detailed meshes for collision with environment -->
+    <link name="${arm_id}_${name}">
+      <visual>
+        <geometry>
+          <mesh filename="package://${description_pkg}/meshes/visual/${name}.dae" />
+        </geometry>
+      </visual>
+      <collision>
+        <geometry>
+          <mesh filename="package://franka_description/meshes/collision/${name}.stl" />
+        </geometry>
+      </collision>
+    </link>
+    <!-- sub-link defining coarse geometries of real robot's internal self-collision -->
+    <link name="${arm_id}_${name}_sc">
+      <xacro:unless value="$(arg gazebo)">
+        <xacro:insert_block name="self_collision_geometries" />
+      </xacro:unless>
+    </link>
+    <!-- fixed joint between both sub-links -->
+    <joint name="${arm_id}_${name}_sc_joint" type="fixed">
+      <parent link="${arm_id}_${name}" />
+      <child link="${arm_id}_${name}_sc" />
+    </joint>
+  </xacro:macro>
   <!-- ========================================================== -->
   <!-- Adds the required tags to simulate one joint in gazebo     -->

Commit message: Distinguish link8 and link8_sc

File: franka_description/robots/arm.xacro (robot description, xacro)
@@ -261,5 +261,6 @@
       <limit effort="12" lower="-2.8973" upper="2.8973" velocity="2.6100"/>
     </joint>
-    <link name="${arm_id}_link8">
+    <link name="${arm_id}_link8"/>
+    <link name="${arm_id}_link8_sc">
       <collision>
         <origin xyz="0.0424 0.0424 -0.0250" rpy="${pi} ${pi/2} ${pi/2}"/>
@@ -286,4 +287,8 @@
       <child link="${arm_id}_link8"/>
     </joint>
+    <joint name="${arm_id}_link8_sc_joint" type="fixed">
+      <parent link="${arm_id}_link8" />
+      <child link="${arm_id}_link8_sc" />
+    </joint>
   </xacro:macro>
 </robot>
