Commit message: FIX: Differentiate between ´<xacro:link>` and `<link>´ in Melodic
The `xacro:` prefix was made mandatory in Noetic, while it Melodic it still
produces a warning. This will mean that plain `<link>` will be expanded to
`<xacro:link>` making the macro recursive =S

Giving the macro a unique name like `panda_link` should fix the problem

File: franka_description/robots/arm.xacro (robot description, xacro)
@@ -11,5 +11,5 @@
       </joint>
     </xacro:unless>
-    <xacro:link arm_id="${arm_id}" name="link0">
+    <xacro:panda_link arm_id="${arm_id}" name="link0">
       <self_collision_geometries>
       <collision>
@@ -32,6 +32,6 @@
       </collision>
       </self_collision_geometries>
-    </xacro:link>
-    <xacro:link arm_id="${arm_id}" name="link1">
+    </xacro:panda_link>
+    <xacro:panda_link arm_id="${arm_id}" name="link1">
       <self_collision_geometries>
       <collision>
@@ -54,5 +54,5 @@
       </collision>
       </self_collision_geometries>
-    </xacro:link>
+    </xacro:panda_link>
     <joint name="${arm_id}_joint1" type="revolute">
       <safety_controller k_position="100.0" k_velocity="40.0" soft_lower_limit="-2.8973" soft_upper_limit="2.8973"/>
@@ -63,5 +63,5 @@
       <limit effort="87" lower="-2.8973" upper="2.8973" velocity="2.1750"/>
     </joint>
-    <xacro:link arm_id="${arm_id}" name="link2">
+    <xacro:panda_link arm_id="${arm_id}" name="link2">
       <self_collision_geometries>
       <collision>
@@ -84,5 +84,5 @@
       </collision>
       </self_collision_geometries>
-    </xacro:link>
+    </xacro:panda_link>
     <joint name="${arm_id}_joint2" type="revolute">
       <safety_controller k_position="100.0" k_velocity="40.0" soft_lower_limit="-1.7628" soft_upper_limit="1.7628"/>
@@ -93,5 +93,5 @@
       <limit effort="87" lower="-1.7628" upper="1.7628" velocity="2.1750"/>
     </joint>
-    <xacro:link arm_id="${arm_id}" name="link3">
+    <xacro:panda_link arm_id="${arm_id}" name="link3">
       <self_collision_geometries>
       <collision>
@@ -114,5 +114,5 @@
       </collision>
       </self_collision_geometries>
-    </xacro:link>
+    </xacro:panda_link>
     <joint name="${arm_id}_joint3" type="revolute">
       <safety_controller k_position="100.0" k_velocity="40.0" soft_lower_limit="-2.8973" soft_upper_limit="2.8973"/>
@@ -123,5 +123,5 @@
       <limit effort="87" lower="-2.8973" upper="2.8973" velocity="2.1750"/>
     </joint>
-    <xacro:link arm_id="${arm_id}" name="link4">
+    <xacro:panda_link arm_id="${arm_id}" name="link4">
       <self_collision_geometries>
       <collision>
@@ -144,5 +144,5 @@
       </collision>
       </self_collision_geometries>
-    </xacro:link>
+    </xacro:panda_link>
     <joint name="${arm_id}_joint4" type="revolute">
       <safety_controller k_position="100.0" k_velocity="40.0" soft_lower_limit="-3.0718" soft_upper_limit="-0.0698"/>
@@ -153,5 +153,5 @@
       <limit effort="87" lower="-3.0718" upper="-0.0698" velocity="2.1750"/>
     </joint>
-    <xacro:link arm_id="${arm_id}" name="link5">
+    <xacro:panda_link arm_id="${arm_id}" name="link5">
       <self_collision_geometries>
       <collision>
@@ -192,5 +192,5 @@
       </collision>
       </self_collision_geometries>
-    </xacro:link>
+    </xacro:panda_link>
     <joint name="${arm_id}_joint5" type="revolute">
       <safety_controller k_position="100.0" k_velocity="40.0" soft_lower_limit="-2.8973" soft_upper_limit="2.8973"/>
@@ -201,5 +201,5 @@
       <limit effort="12" lower="-2.8973" upper="2.8973" velocity="2.6100"/>
     </joint>
-    <xacro:link arm_id="${arm_id}" name="link6">
+    <xacro:panda_link arm_id="${arm_id}" name="link6">
       <self_collision_geometries>
       <collision>
@@ -222,5 +222,5 @@
       </collision>
       </self_collision_geometries>
-    </xacro:link>
+    </xacro:panda_link>
     <joint name="${arm_id}_joint6" type="revolute">
       <safety_controller k_position="100.0" k_velocity="40.0" soft_lower_limit="-0.0175" soft_upper_limit="3.7525"/>
@@ -231,5 +231,5 @@
       <limit effort="12" lower="-0.0175" upper="3.7525" velocity="2.6100"/>
     </joint>
-    <xacro:link arm_id="${arm_id}" name="link7">
+    <xacro:panda_link arm_id="${arm_id}" name="link7">
       <self_collision_geometries>
       <collision>
@@ -252,5 +252,5 @@
       </collision>
       </self_collision_geometries>
-    </xacro:link>
+    </xacro:panda_link>
     <joint name="${arm_id}_joint7" type="revolute">
       <safety_controller k_position="100.0" k_velocity="40.0" soft_lower_limit="-2.8973" soft_upper_limit="2.8973"/>

File: franka_description/robots/hand.xacro (robot description, xacro)
@@ -11,5 +11,5 @@
       </joint>
     </xacro:unless>
-    <xacro:link arm_id="${arm_id}" name="hand">
+    <xacro:panda_link arm_id="${arm_id}" name="hand">
       <self_collision_geometries>
       <collision>
@@ -50,5 +50,5 @@
       </collision>
       </self_collision_geometries>
-    </xacro:link>
+    </xacro:panda_link>
     <!-- Define the hand_tcp frame -->
     <link name="${arm_id}_hand_tcp" />

File: franka_description/robots/utils.xacro (robot description, xacro)
@@ -9,5 +9,5 @@
   <!-- self_collision_geometries:  self <collision> models        -->
   <!-- ========================================================== -->
-  <xacro:macro name="link" params="arm_id name **self_collision_geometries">
+  <xacro:macro name="panda_link" params="arm_id name **self_collision_geometries">
     <!-- sub-link defining detailed meshes for collision with environment -->
     <link name="${arm_id}_${name}">
