Commit message: FIX: `ns` -> `arm_id` in gazebo hand macro

File: franka_description/robots/panda_gazebo.xacro (robot description, xacro)
@@ -258,14 +258,14 @@
     </joint>
   </xacro:macro>
-  <xacro:macro name="hand" params="connected_to:='' ns:='' xyz:='0 0 0' rpy:='0 0 0'">
+  <xacro:macro name="hand" params="arm_id:='panda' connected_to:='' xyz:='0 0 0' rpy:='0 0 0'">
     <xacro:include filename="utils.xacro"/>
     <xacro:unless value="${connected_to == ''}">
-      <joint name="${ns}_hand_joint" type="fixed">
+      <joint name="${arm_id}_hand_joint" type="fixed">
         <parent link="${connected_to}"/>
-        <child link="${ns}_hand"/>
+        <child link="${arm_id}_hand"/>
         <origin xyz="${xyz}" rpy="${rpy}"/>
       </joint>
     </xacro:unless>
-    <link name="${ns}_hand">
+    <link name="${arm_id}_hand">
       <visual>
         <geometry>
@@ -316,5 +316,5 @@
       </collision>
     </xacro:macro>
-    <link name="${ns}_leftfinger">
+    <link name="${arm_id}_leftfinger">
       <xacro:inertia-cylinder mass="15e-3" radius="0.01" h="0.04"/>
       <visual>
@@ -325,5 +325,5 @@
       <xacro:finger-collision sign="+" />
     </link>
-    <link name="${ns}_rightfinger">
+    <link name="${arm_id}_rightfinger">
       <xacro:inertia-cylinder mass="15e-3" radius="0.01" h="0.04"/>
       <visual>
@@ -337,9 +337,9 @@
     <!-- Friction specific material for Rubber/Rubber contact -->
     <!-- See: -->
-    <xacro:gazebo-friction link="${ns}_leftfinger" mu="1.13" />
-    <xacro:gazebo-friction link="${ns}_rightfinger" mu="1.13" />
-    <joint name="${ns}_finger_joint1" type="prismatic">
-      <parent link="${ns}_hand"/>
-      <child link="${ns}_leftfinger"/>
+    <xacro:gazebo-friction link="${arm_id}_leftfinger" mu="1.13" />
+    <xacro:gazebo-friction link="${arm_id}_rightfinger" mu="1.13" />
+    <joint name="${arm_id}_finger_joint1" type="prismatic">
+      <parent link="${arm_id}_hand"/>
+      <child link="${arm_id}_leftfinger"/>
       <origin xyz="0 0 0.0584" rpy="0 0 0"/>
       <axis xyz="0 1 0"/>
@@ -347,12 +347,12 @@
       <dynamics friction="0.0" damping="0.03"/>
     </joint>
-    <joint name="${ns}_finger_joint2" type="prismatic">
-      <parent link="${ns}_hand"/>
-      <child link="${ns}_rightfinger"/>
+    <joint name="${arm_id}_finger_joint2" type="prismatic">
+      <parent link="${arm_id}_hand"/>
+      <child link="${arm_id}_rightfinger"/>
       <origin xyz="0 0 0.0584" rpy="0 0 0"/>
       <axis xyz="0 -1 0"/>
       <limit effort="100" lower="0.0" upper="0.04" velocity="0.2"/>
       <dynamics friction="0.0" damping="0.03"/>
-      <mimic joint="${ns}_finger_joint1" />
+      <mimic joint="${arm_id}_finger_joint1" />
     </joint>
   </xacro:macro>
